File: zotzotzotv3.kicad_pcb (KiCad board)
At the start: 2 copper layers, 77.7 x 57.1 mm, 23 parts, among them J1 OLED, SW1 SW_Push, U1 ProMicro

Commit message: update
Routing:
- net row2: track 142.9 -> 142.4 mm
- net row1: track 122.3 -> 121.8 mm

Commit message: THT update
Parts:
- added Reset: Jumper_2_Open, TestPoint:TestPoint_2Pads_Pitch5.08mm_Drill1.3mm, F.Cu at (122.7, 75.9)
- D1, D2, D3, D4, D5, D6, D7, D8, D9: footprint bevin:D_SOD-123-Pretty -> bevin:D3_TH_nonHybrid; moved to F.Cu
- R1: footprint Resistor_SMD:R_0805_2012Metric -> bevin:R3_TH_nonHybrid; moved to F.Cu
- moved R1 3.04 mm to (107.5, 78.4), turned to 90 degrees
- moved D4 1.35 mm to (132.9, 71.3)
- moved D5 1.35 mm to (151.9, 71.3)
- moved D6 1.35 mm to (171.0, 71.3)
- moved D7 1.35 mm to (132.9, 90.4)
- moved D8 1.35 mm to (151.9, 90.4)
- moved D9 1.35 mm to (171.0, 90.4)
- moved D1 1.35 mm to (132.9, 52.3)
- moved D2 1.35 mm to (151.9, 52.3)
- moved D3 1.35 mm to (171.0, 52.3)
Routing:
- net row2: track 142.4 -> 150.3 mm, vias 3 -> 4
- net Net-(R1-Pad2): track 35.7 -> 42.9 mm, vias 0 -> 1
- net row1: track 121.8 -> 128.8 mm
- net row0: track 101.0 -> 107.9 mm
- net +5V: track 36.8 -> 42.7 mm

Commit message: new graphic
Parts:
- moved G*** 0.40 mm to (115.1, 87.1)
Other:
- board text added: "IEEE x KEEBS @ UCI"

Commit message: update
Routing:
- net Net-(D3-Pad2): track 4.47 -> 3.46 mm
- net Net-(D2-Pad2): track 4.47 -> 3.46 mm
- net Net-(D1-Pad2): track 4.47 -> 3.46 mm
- net Net-(D9-Pad2): track 4.47 -> 3.46 mm
- net Net-(D8-Pad2): track 4.47 -> 3.46 mm
- net Net-(D7-Pad2): track 4.47 -> 3.46 mm
- net Net-(D6-Pad2): track 4.47 -> 3.46 mm
- net Net-(D5-Pad2): track 4.47 -> 3.46 mm
- net Net-(D4-Pad2): track 4.47 -> 3.46 mm
- net row2: track 150.3 -> 149.4 mm, vias 4 -> 3
Changed lines of the file:
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@@
   (segment (start 107.491342 51.89825) (end 108.614156 53.021064) (width 0.25) (layer "B.Cu") (net 8))
   (segment (start 108.907049 80.039143) (end 107.499942 81.44625) (width 0.25) (layer "B.Cu") (net 8))
-  (segment (start 109.199942 54.435277) (end 109.199942 73.74625) (width 0.25) (layer "B.Cu") (net 8))
+  (segment (start 109.199942 54.435277) (end 109.199942 79.332036) (width 0.25) (layer "B.Cu") (net 8))
   (segment (start 116.369942 80.607379) (end 116.369942 78.05625) (width 0.25) (layer "B.Cu") (net 8))
   (segment (start 107.499942 81.44625) (end 115.531071 81.44625) (width 0.25) (layer "B.Cu") (net 8))
-  (segment (start 109.199942 73.74625) (end 109.199942 79.332036) (width 0.25) (layer "B.Cu") (net 8))
   (arc (start 115.531071 81.44625) (mid 115.837218 81.385353) (end 116.096757 81.211935) (width 0.25) (layer "B.Cu") (net 8))
   (arc (start 109.199942 79.332036) (mid 109.123822 79.714719) (end 108.907049 80.039143) (width 0.25) (layer "B.Cu") (net 8))
@@
   (segment (start 109.702442 75.44625) (end 107.499942 75.44625) (width 0.25) (layer "F.Cu") (net 9))
   (via (at 110.112442 75.85625) (size 0.6) (drill 0.4) (layers "F.Cu" "B.Cu") (net 9))
-  (segment (start 122.659942 75.85625) (end 122.709942 75.90625) (width 0.25) (layer "B.Cu") (net 9))
   (segment (start 109.063675 50.930583) (end 107.491342 49.35825) (width 0.25) (layer "B.Cu") (net 9))
   (segment (start 110.012442 75.85625) (end 110.112442 75.85625) (width 0.25) (layer "B.Cu") (net 9))
@@
   (via (at 170.999524 89.30625) (size 0.6) (drill 0.4) (layers "F.Cu" "B.Cu") (net 20))
   (via (at 132.899524 89.30625) (size 0.6) (drill 0.4) (layers "F.Cu" "B.Cu") (net 20))
-  (via (at 107.491342 73.11485) (size 0.6) (drill 0.4) (layers "F.Cu" "B.Cu") (net 20))
   (arc (start 125.998274 43.567324) (mid 125.876481 42.955031) (end 125.529645 42.435953) (width 0.25) (layer "F.Cu") (net 20))
   (arc (start 127.943858 89.30625) (mid 127.255028 89.169233) (end 126.671066 88.779042) (width 0.25) (layer "F.Cu") (net 20))
@@
   (arc (start 113.051827 42.554365) (mid 113.765558 42.077465) (end 114.607462 41.91) (width 0.25) (layer "F.Cu") (net 20))
   (arc (start 125.998274 87.360666) (mid 126.135291 88.049496) (end 126.525482 88.633458) (width 0.25) (layer "F.Cu") (net 20))
-  (segment (start 107.491342 72.21825) (end 107.491342 73.11485) (width 0.25) (layer "B.Cu") (net 20))
   (segment (start 151.949524 89.30625) (end 151.949524 93.00625) (width 0.25) (layer "B.Cu") (net 20))
   (segment (start 170.999524 89.30625) (end 170.999524 93.00625) (width 0.25) (layer "B.Cu") (net 20))
   (segment (start 132.899524 89.30625) (end 132.899524 93.00625) (width 0.25) (layer "B.Cu") (net 20))
   (segment (start 132.899524 49.25625) (end 132.899524 45.795) (width 0.25) (layer "B.Cu") (net 21))
-  (segment (start 132.899524 45.795) (end 132.189524 45.085) (width 0.25) (layer "B.Cu") (net 21))
-  (segment (start 151.949524 45.795) (end 151.239524 45.085) (width 0.25) (layer "B.Cu") (net 22))
   (segment (start 151.949524 49.25625) (end 151.949524 45.795) (width 0.25) (layer "B.Cu") (net 22))
   (segment (start 170.999524 49.25625) (end 170.999524 45.795) (width 0.25) (layer "B.Cu") (net 23))
-  (segment (start 170.999524 45.795) (end 170.289524 45.085) (width 0.25) (layer "B.Cu") (net 23))
-  (segment (start 132.899524 64.845) (end 132.189524 64.135) (width 0.25) (layer "B.Cu") (net 24))
   (segment (start 132.899524 68.30625) (end 132.899524 64.845) (width 0.25) (layer "B.Cu") (net 24))
-  (segment (start 151.949524 64.845) (end 151.239524 64.135) (width 0.25) (layer "B.Cu") (net 25))
   (segment (start 151.949524 68.30625) (end 151.949524 64.845) (width 0.25) (layer "B.Cu") (net 25))
   (segment (start 170.999524 68.30625) (end 170.999524 64.845) (width 0.25) (layer "B.Cu") (net 26))
-  (segment (start 170.999524 64.845) (end 170.289524 64.135) (width 0.25) (layer "B.Cu") (net 26))
-  (segment (start 132.899524 83.895) (end 132.189524 83.185) (width 0.25) (layer "B.Cu") (net 27))
   (segment (start 132.899524 87.35625) (end 132.899524 83.895) (width 0.25) (layer "B.Cu") (net 27))
-  (segment (start 151.949524 83.895) (end 151.239524 83.185) (width 0.25) (layer "B.Cu") (net 28))
   (segment (start 151.949524 87.35625) (end 151.949524 83.895) (width 0.25) (layer "B.Cu") (net 28))
   (segment (start 170.999524 87.35625) (end 170.999524 83.895) (width 0.25) (layer "B.Cu") (net 29))
-  (segment (start 170.999524 83.895) (end 170.289524 83.185) (width 0.25) (layer "B.Cu") (net 29))
   (zone (net 1) (net_name "GND") (layers F&B.Cu) (hatch edge 0.508)
-    (connect_pads yes (clearance 0.22))
+    (connect_pads (clearance 0.22))
     (min_thickness 0.22) (filled_areas_thickness no)
     (fill yes (thermal_gap 0.508) (thermal_bridge_width 0.508))
