File: zotzotzotv3.kicad_sch (KiCad schematic)
At the start: 22 parts, among them J1 OLED, SW1 SW_Push, U1 ProMicro

Commit message: update
Changed lines of the file:
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@@
-    (stroke (width 0) (type default) (color 0 0 0 0))
-  )
-  (wire (pts (xy 153.67 59.69) (xy 153.67 58.42))
     (stroke (width 0) (type default) (color 0 0 0 0))
   )
@@
     (stroke (width 0) (type default) (color 0 0 0 0))
   )
-  (wire (pts (xy 153.67 58.42) (xy 172.72 58.42))
+  (wire (pts (xy 163.83 58.42) (xy 172.72 58.42))
     (stroke (width 0) (type default) (color 0 0 0 0))
   )
@@
     (pin "2")
   )
-  (symbol (lib_id "power:GND") (at 153.67 59.69 0) (unit 1)
-    (in_bom yes) (on_board yes) (fields_autoplaced)
-    (property "Reference" "#PWR0103" (id 0) (at 153.67 66.04 0)
-      (effects (font (size 1.27 1.27)) hide)
-    )
-    (property "Value" "GND" (id 1) (at 153.67 64.77 0))
-    (property "Footprint" "" (id 2) (at 153.67 59.69 0)
-      (effects (font (size 1.27 1.27)) hide)
-    )
-    (property "Datasheet" "" (id 3) (at 153.67 59.69 0)
-      (effects (font (size 1.27 1.27)) hide)
-    )
+  (symbol (lib_id "power:GND") (at 163.83 58.42 270) (unit 1)
+    (in_bom yes) (on_board yes) (fields_autoplaced)
+    (property "Reference" "#PWR0103" (id 0) (at 157.48 58.42 0)
+      (effects (font (size 1.27 1.27)) hide)
+    )
+    (property "Value" "GND" (id 1) (at 160.02 58.4199 90)
+      (effects (font (size 1.27 1.27)) (justify right))
+    )
+    (property "Footprint" "" (id 2) (at 163.83 58.42 0)
+      (effects (font (size 1.27 1.27)) hide)
+    )
+    (property "Datasheet" "" (id 3) (at 163.83 58.42 0)
+      (effects (font (size 1.27 1.27)) hide)
+    )

Commit message: THT update
Parts:
- added JP1: Jumper_2_Open, symbol Jumper:Jumper_2_Open
- D1, D2, D3, D4, D5, D6, D7, D8, D9: footprint bevin:D_SOD-123-Pretty -> bevin:D3_TH_nonHybrid
- R1: footprint Resistor_SMD:R_0805_2012Metric -> bevin:R3_TH_nonHybrid
Connections:
- net GND: now also JP1.2 (B)
- net at R1.2, SW1.1, U1.22 (RST): now also JP1.1 (A)
Changed lines of the file:
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@@
   (junction (at 69.85 57.15) (diameter 0) (color 0 0 0 0)
   )
+  (junction (at 254 58.42) (diameter 0) (color 0 0 0 0)
+  )
   (junction (at 113.03 44.45) (diameter 0) (color 0 0 0 0)
   )
@@
   (junction (at 69.85 82.55) (diameter 0) (color 0 0 0 0)
   )
+  (junction (at 243.84 58.42) (diameter 0) (color 0 0 0 0)
+  )
   (junction (at 87.63 69.85) (diameter 0) (color 0 0 0 0)
   )
@@
     (stroke (width 0) (type default) (color 0 0 0 0))
   )
+  (wire (pts (xy 243.84 58.42) (xy 243.84 66.04))
+    (stroke (width 0) (type default) (color 0 0 0 0))
+  )
   (wire (pts (xy 113.03 38.1) (xy 113.03 44.45))
     (stroke (width 0) (type default) (color 0 0 0 0))
   )
   (wire (pts (xy 254 58.42) (xy 264.16 58.42))
+    (stroke (width 0) (type default) (color 0 0 0 0))
+  )
+  (wire (pts (xy 254 58.42) (xy 254 66.04))
     (stroke (width 0) (type default) (color 0 0 0 0))
   )
@@
       (effects (font (size 1.27 1.27)) (justify right))
     )
-    (property "Footprint" "bevin:D_SOD-123-Pretty" (id 2) (at 95.25 54.61 90)
+    (property "Footprint" "bevin:D3_TH_nonHybrid" (id 2) (at 95.25 54.61 90)
       (effects (font (size 1.27 1.27)) hide)
     )
@@
       (effects (font (size 1.27 1.27)) (justify right))
     )
-    (property "Footprint" "bevin:D_SOD-123-Pretty" (id 2) (at 69.85 54.61 90)
+    (property "Footprint" "bevin:D3_TH_nonHybrid" (id 2) (at 69.85 54.61 90)
       (effects (font (size 1.27 1.27)) hide)
     )
@@
       (effects (font (size 1.27 1.27)) (justify left))
     )
-    (property "Footprint" "Resistor_SMD:R_0805_2012Metric" (id 2) (at 238.252 49.53 90)
+    (property "Footprint" "bevin:R3_TH_nonHybrid" (id 2) (at 238.252 49.53 90)
       (effects (font (size 1.27 1.27)) hide)
     )
@@
       (effects (font (size 1.27 1.27)) (justify right))
     )
-    (property "Footprint" "bevin:D_SOD-123-Pretty" (id 2) (at 120.65 54.61 90)
+    (property "Footprint" "bevin:D3_TH_nonHybrid" (id 2) (at 120.65 54.61 90)
       (effects (font (size 1.27 1.27)) hide)
     )
@@
       (effects (font (size 1.27 1.27)) (justify right))
     )
-    (property "Footprint" "bevin:D_SOD-123-Pretty" (id 2) (at 69.85 105.41 90)
+    (property "Footprint" "bevin:D3_TH_nonHybrid" (id 2) (at 69.85 105.41 90)
       (effects (font (size 1.27 1.27)) hide)
     )
@@
       (effects (font (size 1.27 1.27)) (justify right))
     )
-    (property "Footprint" "bevin:D_SOD-123-Pretty" (id 2) (at 95.25 80.01 90)
+    (property "Footprint" "bevin:D3_TH_nonHybrid" (id 2) (at 95.25 80.01 90)
       (effects (font (size 1.27 1.27)) hide)
     )
@@
       (effects (font (size 1.27 1.27)) (justify right))
     )
-    (property "Footprint" "bevin:D_SOD-123-Pretty" (id 2) (at 69.85 80.01 90)
+    (property "Footprint" "bevin:D3_TH_nonHybrid" (id 2) (at 69.85 80.01 90)
       (effects (font (size 1.27 1.27)) hide)
     )
@@
     (property "Datasheet" "" (id 3) (at 93.345 80.645 0)
       (effects (font (size 1.524 1.524)) hide)
+    )
+    (pin "1")
+    (pin "2")
+  )
+  (symbol (lib_id "Jumper:Jumper_2_Open") (at 248.92 66.04 0) (unit 1)
+    (in_bom yes) (on_board yes) (fields_autoplaced)
+    (property "Reference" "JP1" (id 0) (at 248.92 59.69 0))
+    (property "Value" "Jumper_2_Open" (id 1) (at 248.92 62.23 0))
+    (property "Footprint" "" (id 2) (at 248.92 66.04 0)
+      (effects (font (size 1.27 1.27)) hide)
+    )
+    (property "Datasheet" "~" (id 3) (at 248.92 66.04 0)
+      (effects (font (size 1.27 1.27)) hide)
     )
     (pin "1")
@@
       (effects (font (size 1.27 1.27)) (justify right))
     )
-    (property "Footprint" "bevin:D_SOD-123-Pretty" (id 2) (at 95.25 105.41 90)
+    (property "Footprint" "bevin:D3_TH_nonHybrid" (id 2) (at 95.25 105.41 90)
       (effects (font (size 1.27 1.27)) hide)
     )
@@
       (effects (font (size 1.27 1.27)) (justify right))
     )
-    (property "Footprint" "bevin:D_SOD-123-Pretty" (id 2) (at 120.65 105.41 90)
+    (property "Footprint" "bevin:D3_TH_nonHybrid" (id 2) (at 120.65 105.41 90)
       (effects (font (size 1.27 1.27)) hide)
     )
@@
       (effects (font (size 1.27 1.27)) (justify right))
     )
-    (property "Footprint" "bevin:D_SOD-123-Pretty" (id 2) (at 120.65 80.01 90)
+    (property "Footprint" "bevin:D3_TH_nonHybrid" (id 2) (at 120.65 80.01 90)
       (effects (font (size 1.27 1.27)) hide)
     )
@@
     )
     (path "/0397928a-54e8-4f02-a252-64b74e5478e9"
-      (reference "D1") (unit 1) (value "D_Small") (footprint "bevin:D_SOD-123-Pretty")
+      (reference "D1") (unit 1) (value "D_Small") (footprint "bevin:D3_TH_nonHybrid")
     )
     (path "/01eac853-611f-44a3-8057-3c5c1073461c"
-      (reference "D2") (unit 1) (value "D_Small") (footprint "bevin:D_SOD-123-Pretty")
+      (reference "D2") (unit 1) (value "D_Small") (footprint "bevin:D3_TH_nonHybrid")
     )
     (path "/5ec51d1c-2775-4e10-9c6e-18b0392efef4"
-      (reference "D3") (unit 1) (value "D_Small") (footprint "bevin:D_SOD-123-Pretty")
+      (reference "D3") (unit 1) (value "D_Small") (footprint "bevin:D3_TH_nonHybrid")
     )
     (path "/927b80fb-95ad-49a6-a5ff-9268c39afab5"
-      (reference "D4") (unit 1) (value "D_Small") (footprint "bevin:D_SOD-123-Pretty")
+      (reference "D4") (unit 1) (value "D_Small") (footprint "bevin:D3_TH_nonHybrid")
     )
     (path "/70c5f710-4e29-44aa-a1ed-81c96b4dff24"
-      (reference "D5") (unit 1) (value "D_Small") (footprint "bevin:D_SOD-123-Pretty")
+      (reference "D5") (unit 1) (value "D_Small") (footprint "bevin:D3_TH_nonHybrid")
     )
     (path "/e8154154-493e-45be-962e-dddfd1466bd4"
-      (reference "D6") (unit 1) (value "D_Small") (footprint "bevin:D_SOD-123-Pretty")
+      (reference "D6") (unit 1) (value "D_Small") (footprint "bevin:D3_TH_nonHybrid")
     )
     (path "/64613938-0091-4074-bf9d-add9e344f166"
-      (reference "D7") (unit 1) (value "D_Small") (footprint "bevin:D_SOD-123-Pretty")
+      (reference "D7") (unit 1) (value "D_Small") (footprint "bevin:D3_TH_nonHybrid")
     )
     (path "/dd95ff42-e814-43ae-aec6-057aec2b872a"
-      (reference "D8") (unit 1) (value "D_Small") (footprint "bevin:D_SOD-123-Pretty")
+      (reference "D8") (unit 1) (value "D_Small") (footprint "bevin:D3_TH_nonHybrid")
     )
     (path "/de9b69e4-e379-4880-b39e-810fd7f69495"
-      (reference "D9") (unit 1) (value "D_Small") (footprint "bevin:D_SOD-123-Pretty")
+      (reference "D9") (unit 1) (value "D_Small") (footprint "bevin:D3_TH_nonHybrid")
     )
     (path "/61270030-3c79-4c1e-b0f0-d682ff598773"
       (reference "J1") (unit 1) (value "OLED") (footprint "bevin:OLED_v2")
     )
+    (path "/a4c41e56-d0e3-4c41-87f8-b59ed02daca9"
+      (reference "JP1") (unit 1) (value "Jumper_2_Open") (footprint "TestPoint:TestPoint_2Pads_Pitch5.08mm_Drill1.3mm")
+    )
     (path "/1ad52a9a-40b1-4524-ab02-0871e513e91e"
       (reference "MX1") (unit 1) (value "MX-NoLED") (footprint "bevin:MXOnly-1U-NoLED")
@@
     )
     (path "/03a04b22-3c27-492b-b0e1-8d6cb5563c9a"
-      (reference "R1") (unit 1) (value "10k") (footprint "Resistor_SMD:R_0805_2012Metric")
+      (reference "R1") (unit 1) (value "10k") (footprint "bevin:R3_TH_nonHybrid")
     )
     (path "/0fe9ee7c-30e6-43bc-84ab-3c752b95af67"

Commit message: new graphic
Parts:
- renumbered JP1 to RESET
Changed lines of the file:
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@@
   (symbol (lib_id "Jumper:Jumper_2_Open") (at 248.92 66.04 0) (unit 1)
     (in_bom yes) (on_board yes) (fields_autoplaced)
-    (property "Reference" "JP1" (id 0) (at 248.92 59.69 0))
+    (property "Reference" "RESET" (id 0) (at 248.92 59.69 0))
     (property "Value" "Jumper_2_Open" (id 1) (at 248.92 62.23 0))
     (property "Footprint" "" (id 2) (at 248.92 66.04 0)
@@
       (reference "J1") (unit 1) (value "OLED") (footprint "bevin:OLED_v2")
     )
-    (path "/a4c41e56-d0e3-4c41-87f8-b59ed02daca9"
-      (reference "JP1") (unit 1) (value "Jumper_2_Open") (footprint "TestPoint:TestPoint_2Pads_Pitch5.08mm_Drill1.3mm")
-    )
     (path "/1ad52a9a-40b1-4524-ab02-0871e513e91e"
       (reference "MX1") (unit 1) (value "MX-NoLED") (footprint "bevin:MXOnly-1U-NoLED")
@@
       (reference "R1") (unit 1) (value "10k") (footprint "bevin:R3_TH_nonHybrid")
     )
+    (path "/a4c41e56-d0e3-4c41-87f8-b59ed02daca9"
+      (reference "RESET") (unit 1) (value "Jumper_2_Open") (footprint "TestPoint:TestPoint_2Pads_Pitch5.08mm_Drill1.3mm")
+    )
     (path "/0fe9ee7c-30e6-43bc-84ab-3c752b95af67"

Commit message: annotated
Parts:
- RESET1: renamed from RESET; footprint (none) -> TestPoint:TestPoint_2Pads_Pitch5.08mm_Drill1.3mm
Connections:
- no-connect marks 0 -> 8
Other:
- note added: "OLED"
- note added: "ProMicro Circuit"
- note added: "Reset Circuit"
- note added: "Switch Matrix"
- company: uci keeb club -> keeb club x IEEE club
- moved on the sheet: D1, D2, D3, D4, D5, D6, D7, D8, D9, J1, MX1, MX2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
